File: SuperStation one controller SNAC breakout/SNAC.kicad_sch (KiCad schematic)
At the start: 44 parts, among them J2 USB3_A, J5 Conn_01x09_Pin, J7 Conn_01x09_Pin, Q1 BSS138, Q2 BSS138, Q3 BSS138, Q4 BSS138, Q5 BSS138, Q6 BSS138, Q7 BSS138, SW1 SW_SPST, U1 NCP1117-5.0_SOT223, U2 SN74LVC1G3157, U3 SN74LVC1G3157, U4 SN74LVC1G3157, U5 SN74LVC1G3157, U6 SN74LVC1G3157, U7 SN74LVC1G3157, U8 SN74LVC1G3157

Commit message: added power sheet to schematic and started rough pcb placement
Parts:
- removed C1, C2: 10u, Capacitor_SMD:C_0603_1608Metric, symbol Device:C_Small
- removed JP1: Jumper_2_Open, symbol Jumper:Jumper_2_Open
- removed U1: NCP1117-5.0_SOT223, Package_TO_SOT_SMD:SOT-223-3_TabPin2, symbol Regulator_Linear:NCP1117-5.0_SOT223
- removed unit 2 of U2
- removed unit 2 of U3
- removed unit 2 of U4
- removed unit 2 of U5
- removed unit 2 of U6
- removed unit 2 of U7
- removed unit 2 of U8
- J5: renamed from J7; footprint (none) -> Connector_JST:JST_PH_S8B-PH-SM4-TB_1x08-1MP_P2.00mm_Horizontal
- J6: renamed from J5; footprint (none) -> Connector_JST:JST_PH_S8B-PH-SM4-TB_1x08-1MP_P2.00mm_Horizontal
- JP1: renamed from JP2; footprint (none) -> Jumper:SolderJumper-2_P1.3mm_Bridged_Pad1.0x1.5mm
- JP2: renamed from JP3; footprint (none) -> Jumper:SolderJumper-2_P1.3mm_Bridged_Pad1.0x1.5mm
- JP3: renamed from JP4; footprint (none) -> Jumper:SolderJumper-2_P1.3mm_Bridged_Pad1.0x1.5mm
- JP4: renamed from JP5; footprint (none) -> Jumper:SolderJumper-2_P1.3mm_Bridged_Pad1.0x1.5mm
- JP5: renamed from JP6; footprint (none) -> Jumper:SolderJumper-2_P1.3mm_Bridged_Pad1.0x1.5mm
- JP6: renamed from JP7; footprint (none) -> Jumper:SolderJumper-2_P1.3mm_Bridged_Pad1.0x1.5mm
- JP7: renamed from JP8; footprint (none) -> Jumper:SolderJumper-2_P1.3mm_Bridged_Pad1.0x1.5mm
- U1: renamed from U2; footprint (none) -> Package_TO_SOT_SMD:TSOT-23-6
- U2: renamed from U3; footprint (none) -> Package_TO_SOT_SMD:TSOT-23-6
- U3: renamed from U4; footprint (none) -> Package_TO_SOT_SMD:TSOT-23-6
- U4: renamed from U5; footprint (none) -> Package_TO_SOT_SMD:TSOT-23-6
- U5: renamed from U6; footprint (none) -> Package_TO_SOT_SMD:TSOT-23-6
- U6: renamed from U7; footprint (none) -> Package_TO_SOT_SMD:TSOT-23-6
- U7: renamed from U8; footprint (none) -> Package_TO_SOT_SMD:TSOT-23-6
- renumbered J2 to J7
Connections:
- net D+: now reaches J7.3 (D+), U4.4 (A)
- net MUX_SWITCH: now reaches R15.1, SW1.2 (B), U1.6 (S), U2.6 (S), U3.6 (S), U4.6 (S), U5.6 (S), U6.6 (S), U7.6 (S)
- net D-: now reaches J7.2 (D-), U2.4 (A)
- net RX-: now reaches J7.5 (SSRX-), U6.4 (A)
- net RX+: now reaches J7.6 (SSRX+), U5.4 (A)
- net DRAIN: now reaches J7.7 (DRAIN), U3.4 (A)
- net TX-: now reaches J7.8 (SSTX-), U1.4 (A)
- net TX+: now reaches J7.9 (SSTX+), U7.4 (A)
Other:
- note added: "3.3V AND 5V LOGIC SWITCH"
- note added: "DATA LINE DISCONECTS FOR DEBUGGING"
- note added: "SNAC USB CONNECTOR"
- note removed: "RUMBLE VOLTAGE STEPDOWN DNP REGULATOR AND BRIDGE JUMPER IF RUMBLE VOLTAGE = 5V"
- note removed: "To SNACs"

Commit message: board layout and added debug breakouts for all signals
Parts:
- removed SW1: SW_SPST, symbol Switch:SW_SPST
- added J10, J11: Conn_01x08_Pin, Connector_PinHeader_2.54mm:PinHeader_1x08_P2.54mm_Vertical, symbol Connector:Conn_01x08_Pin
- added J12: Conn_01x02_Pin, Connector_PinHeader_2.54mm:PinHeader_1x02_P2.54mm_Vertical, symbol Connector:Conn_01x02_Pin
- added J13: Conn_01x05_Pin, Connector_PinHeader_2.54mm:PinHeader_1x05_P2.54mm_Vertical, symbol Connector:Conn_01x05_Pin
- J7: renamed from J5; value Conn_01x09_Pin -> JST-PH; footprint Connector_JST:JST_PH_S8B-PH-SM4-TB_1x08-1MP_P2.00mm_Horizontal -> Connector_JST:JST_PH_S9B-PH-SM4-TB_1x09-1MP_P2.00mm_Horizontal; symbol Connector:Conn_01x09_Pin -> Connector_Generic_MountingPin:Conn_01x09_MountingPin
- J8: renamed from J6; value Conn_01x09_Pin -> JST-PH; footprint Connector_JST:JST_PH_S8B-PH-SM4-TB_1x08-1MP_P2.00mm_Horizontal -> Connector_JST:JST_PH_S9B-PH-SM4-TB_1x09-1MP_P2.00mm_Horizontal; symbol Connector:Conn_01x09_Pin -> Connector_Generic_MountingPin:Conn_01x09_MountingPin
- renumbered J7 to J9, JP6 to JP1, JP4 to JP2, JP1 to JP3, JP5 to JP4, JP7 to JP5, JP3 to JP6, JP2 to JP7
Connections:
- net +3.3V: now also J13.2 (Pin_2)
- net +5V: now also R15.2, J13.3 (Pin_3)
- net +7.5V: now also J13.4 (Pin_4)
- net GND: now also J7.MP (MountPin), J8.MP (MountPin), J10.1 (Pin_1), J11.1 (Pin_1), J12.2 (Pin_2), J13.1 (Pin_1); no longer R15.2
- net HV1: now also J11.2 (Pin_2)
- net HV2: now also J11.3 (Pin_3)
- net HV3: now also J11.4 (Pin_4)
- net HV4: now also J11.5 (Pin_5)
- net HV5: now also J11.6 (Pin_6)
- net HV6: now also J11.7 (Pin_7)
- net HV7: now also J11.8 (Pin_8)
- net LV1: now also J10.2 (Pin_2)
- net LV2: now also J10.3 (Pin_3)
- net LV3: now also J10.4 (Pin_4)
- net LV4: now also J10.5 (Pin_5)
- net LV5: now also J10.6 (Pin_6)
- net LV6: now also J10.7 (Pin_7)
- net LV7: now also J10.8 (Pin_8)
- net MUX_SWITCH: now also J12.1 (Pin_1), J13.5 (Pin_5)
Other:
- note added: "3.3V AND 5V LOGIC SWITCH JUMPER 5V = NO JUMPER 3.3V = JUMPER"
- note added: "DEBUG BREAKOUT"
- note removed: "3.3V AND 5V LOGIC SWITCH"
- moved on the sheet: R15

Commit message: completed board layout
Connections:
- net GND: now also J12.1 (Pin_1); no longer J12.2 (Pin_2)
- net MUX_SWITCH: now also J12.2 (Pin_2); no longer J12.1 (Pin_1)
Changed lines of the file:
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@@
+	)
+	(symbol
+		(lib_id "Connector:Conn_01x02_Pin")
+		(at 402.59 208.28 270)
+		(unit 1)
+		(exclude_from_sim no)
+		(in_bom yes)
+		(on_board yes)
+		(dnp no)
+		(property "Reference" "J12"
+			(at 402.336 204.47 90)
+			(effects
+				(font
+					(size 1.27 1.27)
+				)
+				(justify right)
+			)
+		)
+		(property "Value" "Conn_01x02_Pin"
+			(at 410.972 206.756 90)
+			(effects
+				(font
+					(size 1.27 1.27)
+				)
+				(justify right)
+			)
+		)
+		(property "Footprint" "Connector_PinHeader_2.54mm:PinHeader_1x02_P2.54mm_Vertical"
+			(at 402.59 208.28 0)
+			(effects
+				(font
+					(size 1.27 1.27)
+				)
+				(hide yes)
+			)
+		)
+		(property "Datasheet" "~"
+			(at 402.59 208.28 0)
+			(effects
+				(font
+					(size 1.27 1.27)
+				)
+				(hide yes)
+			)
+		)
+		(property "Description" "Generic connector, single row, 01x02, script generated"
+			(at 402.59 208.28 0)
+			(effects
+				(font
+					(size 1.27 1.27)
+				)
+				(hide yes)
+			)
+		)
+		(pin "1"
+		)
+		(pin "2"
+		)
+		(instances
+			(project "SuperStation one controller SNAC breakout"
+				(path "/cbd92933-d20e-42b7-906c-813e5f34c94a/fbfcc61c-380e-426e-8388-ba29034c9159"
+					(reference "J12")
+					(unit 1)
+				)
+			)
+		)
 	)
 	(symbol
@@
 					(unit 1)
 				)
-			)
-		)
-	)
-	(symbol
-		(lib_id "Connector:Conn_01x02_Pin")
-		(at 400.05 208.28 90)
-		(mirror x)
-		(unit 1)
-		(exclude_from_sim no)
-		(in_bom yes)
-		(on_board yes)
-		(dnp no)
-		(property "Reference" "J12"
-			(at 403.86 210.1851 90)
-			(effects
-				(font
-					(size 1.27 1.27)
-				)
-				(justify right)
-			)
-		)
-		(property "Value" "Conn_01x02_Pin"
-			(at 403.352 213.106 90)
-			(effects
-				(font
-					(size 1.27 1.27)
-				)
-				(justify right)
-			)
-		)
-		(property "Footprint" "Connector_PinHeader_2.54mm:PinHeader_1x02_P2.54mm_Vertical"
-			(at 400.05 208.28 0)
-			(effects
-				(font
-					(size 1.27 1.27)
-				)
-				(hide yes)
-			)
-		)
-		(property "Datasheet" "~"
-			(at 400.05 208.28 0)
-			(effects
-				(font
-					(size 1.27 1.27)
-				)
-				(hide yes)
-			)
-		)
-		(property "Description" "Generic connector, single row, 01x02, script generated"
-			(at 400.05 208.28 0)
-			(effects
-				(font
-					(size 1.27 1.27)
-				)
-				(hide yes)
-			)
-		)
-		(pin "1"
-		)
-		(pin "2"
-		)
-		(instances
-			(project ""
-				(path "/cbd92933-d20e-42b7-906c-813e5f34c94a/fbfcc61c-380e-426e-8388-ba29034c9159"
-					(reference "J12")
-					(unit 1)
-				)
