File: SNAC EDU/SNAC.kicad_sch (KiCad schematic)
At the start: 43 parts, among them J10 Conn_01x08_Pin, J11 Conn_01x08_Pin, J12 Conn_01x02_Pin, J13 Conn_01x05_Pin, J7 JST-PH, J8 JST-PH, J9 USB3_A, Q1 BSS138, Q2 BSS138, Q3 BSS138, Q4 BSS138, Q5 BSS138, Q6 BSS138, Q7 BSS138, U1 SN74LVC1G3157, U2 SN74LVC1G3157, U3 SN74LVC1G3157, U4 SN74LVC1G3157, U5 SN74LVC1G3157, U6 SN74LVC1G3157, U7 SN74LVC1G3157

Commit message: split the controller and levelshifter into 2 projects for easier manufacturing
Parts:
- added JP10, JP11, JP12, JP13, JP9: Jumper_2_Bridged, Jumper:SolderJumper-2_P1.3mm_Bridged_Pad1.0x1.5mm, symbol Jumper:Jumper_2_Bridged
- renumbered J7 to J1, J8 to J2, J9 to J3, J10 to J4, J11 to J5, J12 to J6, J13 to J7
Connections:
- net ACK: now also JP9.2 (B); no longer J2.3 (Pin_3)
- net CLK: now also JP11.2 (B); no longer J2.5 (Pin_5)
- net CMD: now also JP12.2 (B); no longer J2.7 (Pin_7)
- net DAT: now also JP13.2 (B); no longer J2.8 (Pin_8)
- net IRQ10: now also JP10.2 (B); no longer J2.4 (Pin_4)
- new net: J2.3 (Pin_3), JP9.1 (A)
- new net: J2.4 (Pin_4), JP10.1 (A)
- new net: J2.5 (Pin_5), JP11.1 (A)
- new net: J2.7 (Pin_7), JP12.1 (A)
- new net: J2.8 (Pin_8), JP13.1 (A)
