File: SNAC EDU/SNAC.kicad_sch (KiCad schematic)
At the start: 46 parts, among them J1 Conn_01x10_MountingPin, J2 USB3_A, J3 Conn_01x08_Pin, J4 Conn_01x08_Pin, J5 Conn_01x05_Pin, J6 Conn_01x02_Pin, Q1 BSS138, Q2 BSS138, Q3 BSS138, Q4 BSS138, Q5 BSS138, Q6 BSS138, Q7 BSS138, U1 SN74LVC1G3157, U2 SN74LVC1G3157, U3 SN74LVC1G3157, U4 SN74LVC1G3157, U5 SN74LVC1G3157, U6 SN74LVC1G3157, U7 SN74LVC1G3157

Commit message: Updated JP refdes
Parts:
- renumbered JP3 to JP1, JP4 to JP2, JP5 to JP3, JP6 to JP4, JP7 to JP5, JP9 to JP6, JP10 to JP7
Connections:
- net +3.3V: now also J5.4 (Pin_4); no longer J5.2 (Pin_2)
- net +7.6V: now also J5.2 (Pin_2); no longer J5.4 (Pin_4)
Changed lines of the file:
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@@
 	)
 	(symbol
+		(lib_id "power:+7.5V")
+		(at 50.8 200.66 0)
+		(mirror y)
+		(unit 1)
+		(body_style 1)
+		(exclude_from_sim no)
+		(in_bom yes)
+		(on_board yes)
+		(in_pos_files yes)
+		(dnp no)
+		(property "Reference" "#PWR024"
+			(at 50.8 204.47 0)
+			(hide yes)
+			(show_name no)
+			(do_not_autoplace no)
+			(effects
+				(font
+					(size 1.27 1.27)
+				)
+			)
+		)
+		(property "Value" "+7.6V"
+			(at 47.498 195.58 0)
+			(show_name no)
+			(do_not_autoplace no)
+			(effects
+				(font
+					(size 1.27 1.27)
+				)
+				(justify right)
+			)
+		)
+		(property "Footprint" ""
+			(at 50.8 200.66 0)
+			(hide yes)
+			(show_name no)
+			(do_not_autoplace no)
+			(effects
+				(font
+					(size 1.27 1.27)
+				)
+			)
+		)
+		(property "Datasheet" ""
+			(at 50.8 200.66 0)
+			(hide yes)
+			(show_name no)
+			(do_not_autoplace no)
+			(effects
+				(font
+					(size 1.27 1.27)
+				)
+			)
+		)
+		(property "Description" "Power symbol creates a global label with name \"+7.5V\""
+			(at 50.8 200.66 0)
+			(hide yes)
+			(show_name no)
+			(do_not_autoplace no)
+			(effects
+				(font
+					(size 1.27 1.27)
+				)
+			)
+		)
+		(pin "1"
+		)
+		(instances
+			(project "SNAC EDU"
+				(path "/cbd92933-d20e-42b7-906c-813e5f34c94a/fbfcc61c-380e-426e-8388-ba29034c9159"
+					(reference "#PWR024")
+					(unit 1)
+				)
+			)
+		)
+	)
+	(symbol
 		(lib_id "power:+3.3V")
 		(at 50.8 30.48 0)
@@
 		(in_pos_files yes)
 		(dnp no)
-		(property "Reference" "JP6"
+		(property "Reference" "JP4"
 			(at 86.36 48.768 0)
 			(show_name no)
@@
 			(project "SNAC EDU"
 				(path "/cbd92933-d20e-42b7-906c-813e5f34c94a/fbfcc61c-380e-426e-8388-ba29034c9159"
-					(reference "JP6")
+					(reference "JP4")
 					(unit 1)
 				)
@@
 		(in_pos_files yes)
 		(dnp no)
-		(property "Reference" "JP7"
+		(property "Reference" "JP5"
 			(at 86.36 51.308 0)
 			(show_name no)
@@
 			(project "SNAC EDU"
 				(path "/cbd92933-d20e-42b7-906c-813e5f34c94a/fbfcc61c-380e-426e-8388-ba29034c9159"
-					(reference "JP7")
+					(reference "JP5")
 					(unit 1)
 				)
@@
 	)
 	(symbol
-		(lib_id "power:+3.3V")
-		(at 50.8 200.66 0)
-		(unit 1)
-		(body_style 1)
-		(exclude_from_sim no)
-		(in_bom yes)
-		(on_board yes)
-		(in_pos_files yes)
-		(dnp no)
-		(fields_autoplaced yes)
-		(property "Reference" "#PWR022"
-			(at 50.8 204.47 0)
-			(hide yes)
-			(show_name no)
-			(do_not_autoplace no)
-			(effects
-				(font
-					(size 1.27 1.27)
-				)
-			)
-		)
-		(property "Value" "+3.3V"
-			(at 50.8 195.58 0)
-			(show_name no)
-			(do_not_autoplace no)
-			(effects
-				(font
-					(size 1.27 1.27)
-				)
-			)
-		)
-		(property "Footprint" ""
-			(at 50.8 200.66 0)
-			(hide yes)
-			(show_name no)
-			(do_not_autoplace no)
-			(effects
-				(font
-					(size 1.27 1.27)
-				)
-			)
-		)
-		(property "Datasheet" ""
-			(at 50.8 200.66 0)
-			(hide yes)
-			(show_name no)
-			(do_not_autoplace no)
-			(effects
-				(font
-					(size 1.27 1.27)
-				)
-			)
-		)
-		(property "Description" "Power symbol creates a global label with name \"+3.3V\""
-			(at 50.8 200.66 0)
-			(hide yes)
-			(show_name no)
-			(do_not_autoplace no)
-			(effects
-				(font
-					(size 1.27 1.27)
-				)
-			)
-		)
-		(pin "1"
-		)
-		(instances
-			(project "SNAC EDU"
-				(path "/cbd92933-d20e-42b7-906c-813e5f34c94a/fbfcc61c-380e-426e-8388-ba29034c9159"
-					(reference "#PWR022")
-					(unit 1)
-				)
-			)
-		)
-	)
-	(symbol
 		(lib_id "power:+5V")
 		(at 57.15 200.66 0)
@@
 		(in_pos_files yes)
 		(dnp no)
-		(property "Reference" "JP3"
+		(property "Reference" "JP1"
 			(at 86.36 41.148 0)
 			(show_name no)
@@
 			(project "SNAC EDU"
 				(path "/cbd92933-d20e-42b7-906c-813e5f34c94a/fbfcc61c-380e-426e-8388-ba29034c9159"
-					(reference "JP3")
+					(reference "JP1")
 					(unit 1)
 				)
@@
 	)
 	(symbol
-		(lib_id "Connector:Conn_01x05_Pin")
-		(at 38.1 210.82 0)
+		(lib_id "power:+3.3V")
+		(at 63.5 200.66 0)
 		(unit 1)
 		(body_style 1)
@@
 		(on_board yes)
 		(in_pos_files yes)
-		(dnp yes)
+		(dnp no)
 		(fields_autoplaced yes)
-		(property "Reference" "J5"
-			(at 38.735 200.66 0)
+		(property "Reference" "#PWR022"
+			(at 63.5 204.47 0)
+			(hide yes)
 			(show_name no)
 			(do_not_autoplace no)
@@
 			)
 		)
-		(property "Value" "Conn_01x05_Pin"
-			(at 38.735 203.2 0)
+		(property "Value" "+3.3V"
+			(at 63.5 195.58 0)
 			(show_name no)
 			(do_not_autoplace no)
@@
 			)
 		)
-		(property "Footprint" "Connector_PinHeader_2.54mm:PinHeader_1x05_P2.54mm_Vertical"
-			(at 38.1 210.82 0)
+		(property "Footprint" ""
+			(at 63.5 200.66 0)
 			(hide yes)
 			(show_name no)
@@
 		)
 		(property "Datasheet" ""
-			(at 38.1 210.82 0)
+			(at 63.5 200.66 0)
 			(hide yes)
 			(show_name no)
@@
 			)
 		)
-		(property "Description" "Generic connector, single row, 01x05, script generated"
-			(at 38.1 210.82 0)
+		(property "Description" "Power symbol creates a global label with name \"+3.3V\""
+			(at 63.5 200.66 0)
 			(hide yes)
 			(show_name no)
@@
 			)
 		)
-		(pin "3"
-		)
-		(pin "2"
-		)
-		(pin "4"
-		)
-		(pin "5"
-		)
 		(pin "1"
 		)
@@
 			(project "SNAC EDU"
 				(path "/cbd92933-d20e-42b7-906c-813e5f34c94a/fbfcc61c-380e-426e-8388-ba29034c9159"
-					(reference "J5")
+					(reference "#PWR022")
 					(unit 1)
 				)
@@
 	)
 	(symbol
-		(lib_id "power:+5V")
-		(at 271.78 74.93 0)
+		(lib_id "Connector:Conn_01x05_Pin")
+		(at 38.1 210.82 0)
 		(unit 1)
 		(body_style 1)
@@
 		(on_board yes)
 		(in_pos_files yes)
-		(dnp no)
+		(dnp yes)
 		(fields_autoplaced yes)
-		(property "Reference" "#PWR08"
-			(at 271.78 78.74 0)
-			(hide yes)
+		(property "Reference" "J5"
+			(at 38.735 200.66 0)
 			(show_name no)
 			(do_not_autoplace no)
@@
 			)
 		)
-		(property "Value" "+5V"
-			(at 271.78 69.85 0)
+		(property "Value" "Conn_01x05_Pin"
+			(at 38.735 203.2 0)
 			(show_name no)
 			(do_not_autoplace no)
@@
 			)
 		)
-		(property "Footprint" ""
-			(at 271.78 74.93 0)
+		(property "Footprint" "Connector_PinHeader_2.54mm:PinHeader_1x05_P2.54mm_Vertical"
+			(at 38.1 210.82 0)
 			(hide yes)
 			(show_name no)
@@
 		)
 		(property "Datasheet" ""
-			(at 271.78 74.93 0)
+			(at 38.1 210.82 0)
 			(hide yes)
 			(show_name no)
@@
 			)
 		)
-		(property "Description" "Power symbol creates a global label with name \"+5V\""
-			(at 271.78 74.93 0)
+		(property "Description" "Generic connector, single row, 01x05, script generated"
+			(at 38.1 210.82 0)
 			(hide yes)
 			(show_name no)
@@
 			)
 		)
+		(pin "3"
+		)
+		(pin "2"
+		)
+		(pin "4"
+		)
+		(pin "5"
+		)
 		(pin "1"
 		)
@@
 			(project "SNAC EDU"
 				(path "/cbd92933-d20e-42b7-906c-813e5f34c94a/fbfcc61c-380e-426e-8388-ba29034c9159"
-					(reference "#PWR08")
+					(reference "J5")
 					(unit 1)
 				)
@@
 	)
 	(symbol
-		(lib_id "power:+7.5V")
-		(at 63.5 200.66 0)
-		(mirror y)
+		(lib_id "power:+5V")
+		(at 271.78 74.93 0)
 		(unit 1)
 		(body_style 1)
@@
 		(in_pos_files yes)
 		(dnp no)
-		(property "Reference" "#PWR024"
-			(at 63.5 204.47 0)
+		(fields_autoplaced yes)
+		(property "Reference" "#PWR08"
+			(at 271.78 78.74 0)
 			(hide yes)
 			(show_name no)
@@
 			)
 		)
-		(property "Value" "+7.6V"
-			(at 60.198 195.58 0)
+		(property "Value" "+5V"
+			(at 271.78 69.85 0)
 			(show_name no)
 			(do_not_autoplace no)
@@
 					(size 1.27 1.27)
 				)
-				(justify right)
 			)
 		)
 		(property "Footprint" ""
-			(at 63.5 200.66 0)
+			(at 271.78 74.93 0)
 			(hide yes)
 			(show_name no)
@@
 		)
 		(property "Datasheet" ""
-			(at 63.5 200.66 0)
+			(at 271.78 74.93 0)
 			(hide yes)
 			(show_name no)
@@
 			)
 		)
-		(property "Description" "Power symbol creates a global label with name \"+7.5V\""
-			(at 63.5 200.66 0)
+		(property "Description" "Power symbol creates a global label with name \"+5V\""
+			(at 271.78 74.93 0)
 			(hide yes)
 			(show_name no)
@@
 			(project "SNAC EDU"
 				(path "/cbd92933-d20e-42b7-906c-813e5f34c94a/fbfcc61c-380e-426e-8388-ba29034c9159"
-					(reference "#PWR024")
+					(reference "#PWR08")
 					(unit 1)
 				)
@@
 		(in_pos_files yes)
 		(dnp no)
-		(property "Reference" "JP5"
+		(property "Reference" "JP3"
 			(at 86.36 46.228 0)
 			(show_name no)
@@
 			(project "SNAC EDU"
 				(path "/cbd92933-d20e-42b7-906c-813e5f34c94a/fbfcc61c-380e-426e-8388-ba29034c9159"
-					(reference "JP5")
+					(reference "JP3")
 					(unit 1)
 				)
@@
 		(in_pos_files yes)
 		(dnp no)
-		(property "Reference" "JP10"
+		(property "Reference" "JP7"
 			(at 86.36 56.388 0)
 			(show_name no)
@@
 			(project "SNAC EDU"
 				(path "/cbd92933-d20e-42b7-906c-813e5f34c94a/fbfcc61c-380e-426e-8388-ba29034c9159"
-					(reference "JP10")
+					(reference "JP7")
 					(unit 1)
 				)
@@
 		(in_pos_files yes)
 		(dnp no)
-		(property "Reference" "JP9"
+		(property "Reference" "JP6"
 			(at 86.36 53.848 0)
 			(show_name no)
@@
 			(project "SNAC EDU"
 				(path "/cbd92933-d20e-42b7-906c-813e5f34c94a/fbfcc61c-380e-426e-8388-ba29034c9159"
-					(reference "JP9")
+					(reference "JP6")
 					(unit 1)
 				)
@@
 		(in_pos_files yes)
 		(dnp no)
-		(property "Reference" "JP4"
+		(property "Reference" "JP2"
 			(at 86.36 43.688 0)
 			(show_name no)
@@
 			(project "SNAC EDU"
 				(path "/cbd92933-d20e-42b7-906c-813e5f34c94a/fbfcc61c-380e-426e-8388-ba29034c9159"
-					(reference "JP4")
+					(reference "JP2")
 					(unit 1)
 				)
