File: SNAC EDU/power.kicad_sch (KiCad schematic)
At the start: 11 parts, among them U1 SN74LVC1G3157, U2 SN74LVC1G3157, U3 SN74LVC1G3157, U4 SN74LVC1G3157, U5 SN74LVC1G3157, U6 SN74LVC1G3157, U7 SN74LVC1G3157, U9 XC6206P332MR

Commit message: split the controller and levelshifter into 2 projects for easier manufacturing
Parts:
- renumbered U9 to U8
Changed lines of the file:
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@@
 		(dnp no)
 		(fields_autoplaced yes)
-		(property "Reference" "#PWR041"
+		(property "Reference" "#PWR029"
 			(at 214.63 53.34 0)
 			(effects
@@
 			(project "SuperStation one controller SNAC breakout"
 				(path "/cbd92933-d20e-42b7-906c-813e5f34c94a/9f4e6185-3dfc-4ab7-b065-b07efc3c4f4a"
-					(reference "#PWR041")
+					(reference "#PWR029")
 					(unit 1)
 				)
@@
 		(dnp no)
 		(fields_autoplaced yes)
-		(property "Reference" "#PWR057"
+		(property "Reference" "#PWR045"
 			(at 66.04 85.09 0)
 			(effects
@@
 			(project "SuperStation one controller SNAC breakout"
 				(path "/cbd92933-d20e-42b7-906c-813e5f34c94a/9f4e6185-3dfc-4ab7-b065-b07efc3c4f4a"
-					(reference "#PWR057")
+					(reference "#PWR045")
 					(unit 1)
 				)
@@
 		(dnp no)
 		(fields_autoplaced yes)
-		(property "Reference" "#PWR049"
+		(property "Reference" "#PWR037"
 			(at 189.23 76.2 0)
 			(effects
@@
 			(project "SuperStation one controller SNAC breakout"
 				(path "/cbd92933-d20e-42b7-906c-813e5f34c94a/9f4e6185-3dfc-4ab7-b065-b07efc3c4f4a"
-					(reference "#PWR049")
+					(reference "#PWR037")
 					(unit 1)
 				)
@@
 		(dnp no)
 		(fields_autoplaced yes)
-		(property "Reference" "U9"
+		(property "Reference" "U8"
 			(at 66.04 62.23 0)
 			(effects
@@
 			(project ""
 				(path "/cbd92933-d20e-42b7-906c-813e5f34c94a/9f4e6185-3dfc-4ab7-b065-b07efc3c4f4a"
-					(reference "U9")
+					(reference "U8")
 					(unit 1)
 				)
@@
 		(dnp no)
 		(fields_autoplaced yes)
-		(property "Reference" "#PWR058"
+		(property "Reference" "#PWR046"
 			(at 87.63 85.09 0)
 			(effects
@@
 			(project "SuperStation one controller SNAC breakout"
 				(path "/cbd92933-d20e-42b7-906c-813e5f34c94a/9f4e6185-3dfc-4ab7-b065-b07efc3c4f4a"
-					(reference "#PWR058")
+					(reference "#PWR046")
 					(unit 1)
 				)
@@
 		(dnp no)
 		(fields_autoplaced yes)
-		(property "Reference" "#PWR047"
+		(property "Reference" "#PWR035"
 			(at 44.45 58.42 0)
 			(effects
@@
 			(project "SuperStation one controller SNAC breakout"
 				(path "/cbd92933-d20e-42b7-906c-813e5f34c94a/9f4e6185-3dfc-4ab7-b065-b07efc3c4f4a"
-					(reference "#PWR047")
+					(reference "#PWR035")
 					(unit 1)
 				)
@@
 		(dnp no)
 		(fields_autoplaced yes)
-		(property "Reference" "#PWR055"
+		(property "Reference" "#PWR043"
 			(at 341.63 76.2 0)
 			(effects
@@
 			(project "SuperStation one controller SNAC breakout"
 				(path "/cbd92933-d20e-42b7-906c-813e5f34c94a/9f4e6185-3dfc-4ab7-b065-b07efc3c4f4a"
-					(reference "#PWR055")
+					(reference "#PWR043")
 					(unit 1)
 				)
@@
 		(dnp no)
 		(fields_autoplaced yes)
-		(property "Reference" "#PWR043"
+		(property "Reference" "#PWR031"
 			(at 265.43 53.34 0)
 			(effects
@@
 			(project "SuperStation one controller SNAC breakout"
 				(path "/cbd92933-d20e-42b7-906c-813e5f34c94a/9f4e6185-3dfc-4ab7-b065-b07efc3c4f4a"
-					(reference "#PWR043")
+					(reference "#PWR031")
 					(unit 1)
 				)
@@
 		(dnp no)
 		(fields_autoplaced yes)
-		(property "Reference" "#PWR048"
+		(property "Reference" "#PWR036"
 			(at 87.63 58.42 0)
 			(effects
@@
 			(project "SuperStation one controller SNAC breakout"
 				(path "/cbd92933-d20e-42b7-906c-813e5f34c94a/9f4e6185-3dfc-4ab7-b065-b07efc3c4f4a"
-					(reference "#PWR048")
+					(reference "#PWR036")
 					(unit 1)
 				)
@@
 		(dnp no)
 		(fields_autoplaced yes)
-		(property "Reference" "#PWR042"
+		(property "Reference" "#PWR030"
 			(at 240.03 53.34 0)
 			(effects
@@
 			(project "SuperStation one controller SNAC breakout"
 				(path "/cbd92933-d20e-42b7-906c-813e5f34c94a/9f4e6185-3dfc-4ab7-b065-b07efc3c4f4a"
-					(reference "#PWR042")
+					(reference "#PWR030")
 					(unit 1)
 				)
@@
 		(dnp no)
 		(fields_autoplaced yes)
-		(property "Reference" "#PWR053"
+		(property "Reference" "#PWR041"
 			(at 290.83 76.2 0)
 			(effects
@@
 			(project "SuperStation one controller SNAC breakout"
 				(path "/cbd92933-d20e-42b7-906c-813e5f34c94a/9f4e6185-3dfc-4ab7-b065-b07efc3c4f4a"
-					(reference "#PWR053")
+					(reference "#PWR041")
 					(unit 1)
 				)
@@
 		(dnp no)
 		(fields_autoplaced yes)
-		(property "Reference" "#PWR054"
+		(property "Reference" "#PWR042"
 			(at 316.23 76.2 0)
 			(effects
@@
 			(project "SuperStation one controller SNAC breakout"
 				(path "/cbd92933-d20e-42b7-906c-813e5f34c94a/9f4e6185-3dfc-4ab7-b065-b07efc3c4f4a"
-					(reference "#PWR054")
+					(reference "#PWR042")
 					(unit 1)
 				)
@@
 		(dnp no)
 		(fields_autoplaced yes)
-		(property "Reference" "#PWR056"
+		(property "Reference" "#PWR044"
 			(at 44.45 85.09 0)
 			(effects
@@
 			(project "SuperStation one controller SNAC breakout"
 				(path "/cbd92933-d20e-42b7-906c-813e5f34c94a/9f4e6185-3dfc-4ab7-b065-b07efc3c4f4a"
-					(reference "#PWR056")
+					(reference "#PWR044")
 					(unit 1)
 				)
@@
 		(dnp no)
 		(fields_autoplaced yes)
-		(property "Reference" "#PWR045"
+		(property "Reference" "#PWR033"
 			(at 316.23 53.34 0)
 			(effects
@@
 			(project "SuperStation one controller SNAC breakout"
 				(path "/cbd92933-d20e-42b7-906c-813e5f34c94a/9f4e6185-3dfc-4ab7-b065-b07efc3c4f4a"
-					(reference "#PWR045")
+					(reference "#PWR033")
 					(unit 1)
 				)
@@
 		(dnp no)
 		(fields_autoplaced yes)
-		(property "Reference" "#PWR040"
+		(property "Reference" "#PWR028"
 			(at 189.23 53.34 0)
 			(effects
@@
 			(project "SuperStation one controller SNAC breakout"
 				(path "/cbd92933-d20e-42b7-906c-813e5f34c94a/9f4e6185-3dfc-4ab7-b065-b07efc3c4f4a"
-					(reference "#PWR040")
+					(reference "#PWR028")
 					(unit 1)
 				)
@@
 		(dnp no)
 		(fields_autoplaced yes)
-		(property "Reference" "#PWR052"
+		(property "Reference" "#PWR040"
 			(at 265.43 76.2 0)
 			(effects
@@
 			(project "SuperStation one controller SNAC breakout"
 				(path "/cbd92933-d20e-42b7-906c-813e5f34c94a/9f4e6185-3dfc-4ab7-b065-b07efc3c4f4a"
-					(reference "#PWR052")
+					(reference "#PWR040")
 					(unit 1)
 				)
@@
 		(dnp no)
 		(fields_autoplaced yes)
-		(property "Reference" "#PWR046"
+		(property "Reference" "#PWR034"
 			(at 341.63 53.34 0)
 			(effects
@@
 			(project "SuperStation one controller SNAC breakout"
 				(path "/cbd92933-d20e-42b7-906c-813e5f34c94a/9f4e6185-3dfc-4ab7-b065-b07efc3c4f4a"
-					(reference "#PWR046")
+					(reference "#PWR034")
 					(unit 1)
 				)
@@
 		(dnp no)
 		(fields_autoplaced yes)
-		(property "Reference" "#PWR051"
+		(property "Reference" "#PWR039"
 			(at 240.03 76.2 0)
 			(effects
@@
 			(project "SuperStation one controller SNAC breakout"
 				(path "/cbd92933-d20e-42b7-906c-813e5f34c94a/9f4e6185-3dfc-4ab7-b065-b07efc3c4f4a"
-					(reference "#PWR051")
+					(reference "#PWR039")
 					(unit 1)
 				)
@@
 		(dnp no)
 		(fields_autoplaced yes)
-		(property "Reference" "#PWR044"
+		(property "Reference" "#PWR032"
 			(at 290.83 53.34 0)
 			(effects
@@
 			(project "SuperStation one controller SNAC breakout"
 				(path "/cbd92933-d20e-42b7-906c-813e5f34c94a/9f4e6185-3dfc-4ab7-b065-b07efc3c4f4a"
-					(reference "#PWR044")
+					(reference "#PWR032")
 					(unit 1)
 				)
@@
 		(dnp no)
 		(fields_autoplaced yes)
-		(property "Reference" "#PWR050"
+		(property "Reference" "#PWR038"
 			(at 214.63 76.2 0)
 			(effects
@@
 			(project "SuperStation one controller SNAC breakout"
 				(path "/cbd92933-d20e-42b7-906c-813e5f34c94a/9f4e6185-3dfc-4ab7-b065-b07efc3c4f4a"
-					(reference "#PWR050")
-					(unit 1)
-				)
+					(reference "#PWR038")
+					(unit 1)
+				)
