File: SNAC EDU/power.kicad_sch (KiCad schematic)
At the start: 11 parts, among them U1 SN74LVC1G3157, U2 SN74LVC1G3157, U3 SN74LVC1G3157, U4 SN74LVC1G3157, U5 SN74LVC1G3157, U6 SN74LVC1G3157, U7 SN74LVC1G3157, U8 XC6206P332MR

Commit message: Made schematic notations clearer
Other:
- note added: "MUX POWER"

Commit message: renamed PS1 files to PSX
Parts:
- JP8: now left out of the parts list
Other:
- note added: "ANALOG SWITCH POWER"
- note removed: "MUX POWER"
Changed lines of the file:
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@@
 		)
 	)
-	(text "MUX POWER"
+	(text "ANALOG SWITCH POWER"
 		(exclude_from_sim no)
 		(at 271.272 36.576 0)
@@
 		(body_style 1)
 		(exclude_from_sim yes)
-		(in_bom yes)
-		(on_board yes)
-		(in_pos_files yes)
+		(in_bom no)
+		(on_board yes)
+		(in_pos_files yes)

Commit message: continued routing
Connections:
- net +7.5V renamed +7.6V
Changed lines of the file:
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@@
 			)
 		)
-		(property "Value" "+7.5V"
-			(at 44.45 49.53 0)
+		(property "Value" "+7.6V"
+			(at 46.99 53.3399 0)
 			(show_name no)
 			(do_not_autoplace no)
@@
 					(size 1.27 1.27)
 				)
+				(justify right)
 			)
 		)
