File: SNAC EDU/SNAC EDU.kicad_pcb (KiCad board)
At the start: 2 copper layers, 60 x 50 mm, 52 parts, among them J1 JST-PH, J2 JST-PH, J3 USB3_A, J4 Conn_01x08_Pin, J5 Conn_01x08_Pin, J6 Conn_01x02_Pin, J7 Conn_01x05_Pin, Q1 BSS138, Q2 BSS138, Q3 BSS138, Q4 BSS138, Q5 BSS138, Q6 BSS138, Q7 BSS138, U1 SN74LVC1G3157, U2 SN74LVC1G3157, U3 SN74LVC1G3157, U4 SN74LVC1G3157, U5 SN74LVC1G3157, U6 SN74LVC1G3157, U7 SN74LVC1G3157, U8 XC6206P332MR

Commit message: updated PCBs for JLCs new erial numbering system
Other:
- board text added: "SSONE SNAC EDU v1"
- board text removed: "JLCJLCJLCJLC"

Commit message: started layout
Parts:
- removed J7: Conn_01x05_Pin, Connector_PinHeader_2.54mm:PinHeader_1x05_P2.54mm_Vertical
- removed JP1, JP11, JP12, JP13, JP2: Jumper_2_Bridged, Jumper:SolderJumper-2_P1.3mm_Bridged_Pad1.0x1.5mm
- added D1: LED, LED_SMD:LED_0603_1608Metric, F.Cu at (138.4, 81.8)
- added D2: LED, LED_SMD:LED_0603_1608Metric, F.Cu at (138.4, 84.4)
- added R16: 220, Resistor_SMD:R_0603_1608Metric, F.Cu at (142.7, 81.5)
- added R17: 220, Resistor_SMD:R_0603_1608Metric, F.Cu at (142.7, 84.0)
- J1: value JST-PH -> Conn_01x10_MountingPin; footprint Connector_JST:JST_PH_S9B-PH-SM4-TB_1x09-1MP_P2.00mm_Horizontal -> Connector_JST:JST_PH_S10B-PH-SM4-TB_1x10-1MP_P2.00mm_Horizontal
- J2: value JST-PH -> USB3_A; footprint Connector_JST:JST_PH_S9B-PH-SM4-TB_1x09-1MP_P2.00mm_Horizontal -> Connector_USB:USB3_A_Receptacle_Wuerth_692122030100
- J3: value USB3_A -> Conn_01x08_Pin; footprint Connector_USB:USB3_A_Receptacle_Wuerth_692122030100 -> Connector_PinHeader_2.54mm:PinHeader_1x08_P2.54mm_Vertical
- J5: value Conn_01x08_Pin -> Conn_01x05_Pin; footprint Connector_PinHeader_2.54mm:PinHeader_1x08_P2.54mm_Vertical -> Connector_PinHeader_2.54mm:PinHeader_1x05_P2.54mm_Vertical
- JP10, JP9: moved to F.Cu
- moved J3 183.0 mm to (31.2, 25.3), turned to 0 degrees
- moved J5 149.6 mm to (23.2, 34.0), turned to 0 degrees
- moved J4 139.5 mm to (35.8, 25.3), turned to 0 degrees
- moved C1 86.8 mm to (106.0, 76.8)
- moved C2 82.2 mm to (106.0, 79.3), turned to 0 degrees
- moved JP8 80.1 mm to (110.1, 81.8), turned to 0 degrees
- moved U8 79.4 mm to (110.5, 77.8)
- moved U1 52.6 mm to (139.0, 95.0)
- moved R14 51.4 mm to (134.9, 98.2)
- moved R13 51.4 mm to (128.8, 99.2)
- moved Q7 51.3 mm to (132.0, 99.0)
- moved R15 50.9 mm to (137.6, 75.7)
- moved J6 48.1 mm to (142.6, 74.5), turned to 0 degrees
- moved R5 44.9 mm to (128.8, 94.2)
- moved R6 44.9 mm to (134.9, 93.2)
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Connections:
- J1 pad 1: +3.3V -> +7.5V
- J1 pad 2: +7.5V -> +3.3V
- J1 pad 3: /SNAC/ACK -> /SNAC/ATT1
- J1 pad 4: /SNAC/IRQ10 -> /SNAC/ATT2
- J1 pad 6: /SNAC/ATT1 -> /SNAC/DAT
- J1 pad 7: /SNAC/CMD -> /SNAC/ACK
- J1 pad 8: /SNAC/DAT -> /SNAC/CMD
- J1 pad 9: GND -> /SNAC/IRQ10
- J2 pad 1: +3.3V -> +5V
- J2 pad 2: +7.5V -> /SNAC/SNAC2
- J2 pad 3: Net-(J2-Pin_3) -> /SNAC/SNAC4
- J2 pad 4: Net-(J2-Pin_4) -> GND
- J2 pad 5: Net-(J2-Pin_5) -> /SNAC/SNAC6
- J2 pad 6: /SNAC/ATT2 -> /SNAC/SNAC5
- J2 pad 7: Net-(J2-Pin_7) -> /SNAC/SNAC3
- J2 pad 8: Net-(J2-Pin_8) -> /SNAC/SNAC1
- J2 pad 9: GND -> /SNAC/SNAC7
- J3 pad 1: +5V -> GND
- J3 pad 2: /SNAC/D- -> /SNAC/LV1
- J3 pad 3: /SNAC/D+ -> /SNAC/LV2
- J3 pad 4: GND -> /SNAC/LV3
- J3 pad 5: /SNAC/RX- -> /SNAC/LV4
- J3 pad 6: /SNAC/RX+ -> /SNAC/LV5
- J3 pad 7: /SNAC/DRAIN -> /SNAC/LV6
- J3 pad 8: /SNAC/TX- -> /SNAC/LV7
- J4 pad 2: /SNAC/LV1 -> /SNAC/HV1
- J4 pad 3: /SNAC/LV2 -> /SNAC/HV2
- J4 pad 4: /SNAC/LV3 -> /SNAC/HV3
- J4 pad 5: /SNAC/LV4 -> /SNAC/HV4
- J4 pad 6: /SNAC/LV5 -> /SNAC/HV5
- J4 pad 7: /SNAC/LV6 -> /SNAC/HV6
- J4 pad 8: /SNAC/LV7 -> /SNAC/HV7
- J5 pad 2: /SNAC/HV1 -> +3.3V
- J5 pad 3: /SNAC/HV2 -> +5V
- J5 pad 4: /SNAC/HV3 -> +7.5V
- J5 pad 5: /SNAC/HV4 -> /SNAC/MUX_SWITCH
- JP10 pad 1: Net-(J2-Pin_4) -> /SNAC/IRQ10
- JP10 pad 2: /SNAC/IRQ10 -> /SNAC/LV7
- JP3 pad 1: /SNAC/ACK -> /SNAC/ATT1
- JP3 pad 2: /SNAC/LV3 -> /SNAC/LV2
- JP4 pad 1: /SNAC/CMD -> /SNAC/ATT2
- JP5 pad 1: /SNAC/ATT2 -> /SNAC/CLK
- JP5 pad 2: /SNAC/LV5 -> /SNAC/LV6
- JP6 pad 1: /SNAC/CLK -> /SNAC/DAT
- JP6 pad 2: /SNAC/LV6 -> /SNAC/LV5
- JP7 pad 1: /SNAC/IRQ10 -> /SNAC/ACK
- JP7 pad 2: /SNAC/LV7 -> /SNAC/LV3
- JP9 pad 1: Net-(J2-Pin_3) -> /SNAC/CMD
- JP9 pad 2: /SNAC/ACK -> /SNAC/LV1
- Q2 pad 2: /SNAC/LV2 -> /SNAC/LV5
- Q2 pad 3: /SNAC/HV2 -> /SNAC/HV5
- Q3 pad 2: /SNAC/LV3 -> /SNAC/LV2
- Q3 pad 3: /SNAC/HV3 -> /SNAC/HV2
- Q4 pad 2: /SNAC/LV4 -> /SNAC/LV3
- Q4 pad 3: /SNAC/HV4 -> /SNAC/HV3
- Q5 pad 2: /SNAC/LV5 -> /SNAC/LV7
- Q5 pad 3: /SNAC/HV5 -> /SNAC/HV7
- Q7 pad 2: /SNAC/LV7 -> /SNAC/LV4
- Q7 pad 3: /SNAC/HV7 -> /SNAC/HV4
- R10 pad 2: /SNAC/HV5 -> /SNAC/HV7
- R13 pad 2: /SNAC/LV7 -> /SNAC/LV4
- R14 pad 2: /SNAC/HV7 -> /SNAC/HV4
- R3 pad 2: /SNAC/LV2 -> /SNAC/LV5
- R4 pad 2: /SNAC/HV2 -> /SNAC/HV5
- R5 pad 2: /SNAC/LV3 -> /SNAC/LV2
- R6 pad 2: /SNAC/HV3 -> /SNAC/HV2
- R7 pad 2: /SNAC/LV4 -> /SNAC/LV3
- R8 pad 2: /SNAC/HV4 -> /SNAC/HV3
- R9 pad 2: /SNAC/LV5 -> /SNAC/LV7
- U1 pad 1: /SNAC/HV1 -> /SNAC/HV2
- U1 pad 3: /SNAC/LV1 -> /SNAC/LV2
- U1 pad 4: /SNAC/TX- -> /SNAC/SNAC2
- U2 pad 1: /SNAC/HV2 -> /SNAC/HV4
- U2 pad 3: /SNAC/LV2 -> /SNAC/LV4
- U2 pad 4: /SNAC/D- -> /SNAC/SNAC4
- U3 pad 1: /SNAC/HV3 -> /SNAC/HV6
- U3 pad 3: /SNAC/LV3 -> /SNAC/LV6
- U3 pad 4: /SNAC/DRAIN -> /SNAC/SNAC6
- U4 pad 1: /SNAC/HV4 -> /SNAC/HV5
- U4 pad 3: /SNAC/LV4 -> /SNAC/LV5
- U4 pad 4: /SNAC/D+ -> /SNAC/SNAC5
- U5 pad 1: /SNAC/HV5 -> /SNAC/HV1
- U5 pad 3: /SNAC/LV5 -> /SNAC/LV1
- U5 pad 4: /SNAC/RX+ -> /SNAC/SNAC1
- U6 pad 1: /SNAC/HV6 -> /SNAC/HV7
- U6 pad 3: /SNAC/LV6 -> /SNAC/LV7
- U6 pad 4: /SNAC/RX- -> /SNAC/SNAC7
- U7 pad 1: /SNAC/HV7 -> /SNAC/HV3
- U7 pad 3: /SNAC/LV7 -> /SNAC/LV3
- U7 pad 4: /SNAC/TX+ -> /SNAC/SNAC3
Routing:
- net +3.3V: track 162.8 -> 16.9 mm, vias 9 -> 0
- net +5V: track 141.8 -> 0.00 mm, vias 15 -> 0
- net +7.5V: track 97.8 -> 0.00 mm, vias 2 -> 0
- net /SNAC/LV7: track 88.7 -> 21.4 mm, vias 3 -> 0
- net /SNAC/MUX_SWITCH: track 62.3 -> 0.00 mm, vias 7 -> 0
- net /SNAC/LV1: track 71.1 -> 19.5 mm, vias 4 -> 0
- net /SNAC/LV3: track 67.2 -> 17.4 mm, vias 3 -> 0
- net /SNAC/HV7: track 51.8 -> 4.95 mm, vias 1 -> 0
- net /SNAC/LV2: track 68.1 -> 22.3 mm, vias 4 -> 0
- net /SNAC/LV4: track 65.3 -> 19.6 mm, vias 4 -> 0
- net /SNAC/LV5: track 61.9 -> 16.5 mm, vias 4 -> 0
- net /SNAC/LV6: track 59.2 -> 17.6 mm, vias 2 -> 0
- net /SNAC/HV1: track 40.9 -> 4.95 mm, vias 1 -> 0
- net /SNAC/HV2: track 37.8 -> 4.95 mm, vias 1 -> 0
- net /SNAC/HV3: track 35.0 -> 4.85 mm, vias 1 -> 0
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- removed copper zone on B.Cu, net GND
- removed copper zone on F.Cu, net GND
Other:
- board size 60 x 50 mm -> 100 x 100 mm
- board text removed: "1"
- board text removed: "2"
- board text removed: "3"
- board text removed: "4"
- board text removed: "5"
- board text removed: "6"
- board text removed: "7"
- board text removed: "G"
- board text removed: "HV"
- board text removed: "LV"
- board text removed: "OPEN = 5V CLOSED = 3.3V"
- board text removed: "P1"
- board text removed: "P2"

Commit message: continued routing
Parts:
- moved J4 147.2 mm to (137.9, 131.2), turned to 90 degrees
- moved J3 133.1 mm to (111.7, 131.3), turned to 90 degrees
- moved J5 110.3 mm to (120.2, 86.6), turned to 90 degrees
- moved J6 20.7 mm to (154.1, 91.7), turned to -90 degrees
- moved D2 20.7 mm to (155.8, 95.5), turned to 180 degrees
- moved C1 19.6 mm to (114.3, 94.5)
- moved D1 18.5 mm to (155.7, 88.2), turned to 180 degrees
- moved R17 15.0 mm to (152.4, 95.5), turned to 180 degrees
- moved R15 14.8 mm to (140.2, 90.3), turned to 90 degrees
- moved U8 14.1 mm to (113.5, 91.5), turned to -90 degrees
- moved R16 11.6 mm to (152.2, 88.2)
- moved C2 11.5 mm to (113.3, 88.2)
- moved JP8 10.3 mm to (110.0, 92.0), turned to 90 degrees
- moved J2 0.70 mm to (158.0, 109.1)
Connections:
- net +7.5V renamed +7.6V
Routing:
- net /SNAC/SNAC2: track 0.00 -> 20.4 mm, vias 0 -> 2
- net /SNAC/SNAC4: track 0.00 -> 14.7 mm, vias 0 -> 2
- net +7.6V: track 0.00 -> 11.0 mm
- net +5V: track 0.00 -> 7.38 mm
- net /SNAC/SNAC3: track 12.5 -> 13.1 mm
- net /SNAC/SNAC7: track 17.1 -> 17.8 mm
Other:
- board size 100 x 100 mm -> 60.9 x 51.1 mm

Commit message: Layout and routing progress
Parts:
- moved D2 5.12 mm to (150.7, 95.0)
- moved D1 5.12 mm to (150.6, 87.7)
- moved J6 5.12 mm to (149.0, 91.2)
- moved R16 5.12 mm to (147.1, 87.7)
- moved R17 5.12 mm to (147.3, 95.0)
- moved JP8 1.50 mm to (110.0, 90.5)
- moved R15 0.42 mm to (140.2, 89.9)
- renumbered JP3 to JP1, JP4 to JP2, JP5 to JP3, JP6 to JP4, JP7 to JP5, JP9 to JP6, JP10 to JP7
Connections:
- J5 pad 2: +3.3V -> +7.6V
- J5 pad 4: +7.6V -> +3.3V
Routing:
- net +5V: track 7.38 -> 178.4 mm, vias 0 -> 15
- net /SNAC/MUX_SWITCH: track 0.00 -> 72.6 mm, vias 0 -> 7
- net +3.3V: track 16.9 -> 82.7 mm, vias 0 -> 7
- net /SNAC/LV2: track 22.3 -> 54.4 mm, vias 0 -> 1
- net /SNAC/LV4: track 19.6 -> 48.1 mm, vias 0 -> 1
- net /SNAC/LV6: track 17.6 -> 44.1 mm, vias 0 -> 1
- net /SNAC/LV5: track 16.5 -> 38.6 mm, vias 0 -> 1
- net /SNAC/LV3: track 17.4 -> 38.5 mm, vias 0 -> 1
- net /SNAC/LV1: track 19.5 -> 39.5 mm, vias 0 -> 1
- net +7.6V: track 11.0 -> 25.8 mm
- net /SNAC/LV7: track 21.4 -> 28.8 mm, vias 0 -> 1
- net Net-(D1-A): track 0.00 -> 1.89 mm
- net Net-(D2-A): track 0.00 -> 1.79 mm
- net /SNAC/SNAC1: track 15.3 -> 16.6 mm
- net /SNAC/SNAC7: track 17.8 -> 18.3 mm
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- added copper zone on B.Cu, net GND
- added copper zone on F.Cu, net GND
